File: ZX Diagnostic 2021/ZX Diagnostic 2021.sch (KiCad schematic (older format))
At the start: 29 parts, among them J1 Cartridge, M1 Mounting, M2 Mounting, M3 Mounting, M4 Mounting, U1 27C512, U2 74HCT373

Commit message: Made 74ls245 open collector instead of using resistors
Parts:
- U2: value 74HCT373 -> 74HCT374; symbol 74xx:74HCT373 -> 74xx:74HCT374
Changed lines of the file:
@@
 $EndComp
 $Comp
-L 74xx:74HCT373 U2
+L 74xx:74HCT374 U2
 U 1 1 607A4A1E
 P 3275 2200
 F 0 "U2" H 3050 2850 50  0000 C CNN
-F 1 "74HCT373" V 3275 2200 50  0000 C CNN
+F 1 "74HCT374" V 3275 2200 50  0000 C CNN
 F 2 "Package_DIP:DIP-20_W7.62mm_Socket_LongPads" H 3275 2200 50  0001 C CNN
 F 3 "https://www.ti.com/lit/ds/symlink/sn74hct373.pdf" H 3275 2200 50  0001 C CNN
