File: ZX Cartridge 1983/ZX Cartridge 1983.kicad_pcb (KiCad board)
At the start: 2 copper layers, 57.9 x 61.6 mm, 19 parts, among them J1 Cartridge, M1 Mounting, M2 Mounting, M3 Mounting, M4 Mounting, SW1 ROM_SEL, U1 27C020, U2 MC14495P1

Commit message: Changed 1983 to 1.983
Other:
- board text added: "ZX Cartridge 1.983 github.com/tebl"
- board text removed: "ZX Cartridge 2.021 github.com/tebl"
