File: faceplates/ZX Cartridge 2021 FA1/ZX Cartridge 2021 FA1.kicad_pcb (KiCad board)
At the start: 2 copper layers, 57.9 x 58.9 mm, 11 parts, among them M1 Mounting, M2 Mounting, M3 Mounting, M4 Mounting

Commit message: Larger writable area
Parts:
- removed the sinclair_keyboard_large at (124.3, 87.2)
- removed the sinclair_keyboard_large at (124.3, 83.7)
- added sinclair_keyboard_large: Val**, artwork:cartridge_title_empty2, F.Cu at (124.3, 79.1)
- added sinclair_keyboard_large: Val**, artwork:cartridge_title_empty2, F.Cu at (124.3, 83.9)
- added sinclair_keyboard_large: Val**, artwork:cartridge_title_empty2, F.Cu at (124.3, 86.0)
- added sinclair_keyboard_large: Val**, artwork:cartridge_title_empty2, F.Cu at (124.3, 88.5)
- added sinclair_keyboard_large: Val**, artwork:cartridge_title_empty2, F.Cu at (124.3, 82.2)
- moved sinclair_keyboard_large 0.51 mm to (124.3, 79.6)

Commit message: Changed FA1 design
Parts:
- removed the sinclair_keyboard_large at (124.3, 67.9)
- sinclair_title: footprint artwork:sinclair_title -> artwork:cartridge_label
- moved sinclair_title 4.50 mm to (132.3, 60.3)
- moved sinclair_keyboard_large 0.51 mm to (124.3, 88.0)
